Commit message: added sensor plugins and gz bridge

File: skid_steer_robot_description/urdf/skid_steer_robot.xacro (robot description, xacro)
@@ -2,5 +2,5 @@
 <robot name="skid_steer_robot" xmlns:xacro="http://www.ros.org/wiki/xacro">
 <xacro:include filename="$(find skid_steer_robot_description)/urdf/materials.xacro" />
-<xacro:include filename="$(find skid_steer_robot_description)/urdf/skid_steer_robot.trans" />
+<xacro:include filename="$(find skid_steer_robot_description)/urdf/skid_steer_robot.gazebo" />
 <link name="base_link">
   <inertial>
@@ -23,5 +23,5 @@
   </collision>
 </link>
-<link name="lidar_1">
+<link name="lidar">
   <inertial>
     <origin xyz="-0.008294099570319555 1.386446543170201e-07 0.09520087611989277" rpy="0 0 0"/>
@@ -32,5 +32,5 @@
     <origin xyz="0.08075 -0.000295 -0.109022" rpy="0 0 0"/>
     <geometry>
-      <mesh filename="file://$(find skid_steer_robot_description)/meshes/lidar_1.stl" scale="0.001 0.001 0.001"/>
+      <mesh filename="file://$(find skid_steer_robot_description)/meshes/lidar.stl" scale="0.001 0.001 0.001"/>
     </geometry>
     <material name="steel_satin"/>
@@ -39,9 +39,9 @@
     <origin xyz="0.08075 -0.000295 -0.109022" rpy="0 0 0"/>
     <geometry>
-      <mesh filename="file://$(find skid_steer_robot_description)/meshes/lidar_1.stl" scale="0.001 0.001 0.001"/>
-    </geometry>
-  </collision>
-</link>
-<link name="imu_1">
+      <mesh filename="file://$(find skid_steer_robot_description)/meshes/lidar.stl" scale="0.001 0.001 0.001"/>
+    </geometry>
+  </collision>
+</link>
+<link name="imu">
   <inertial>
     <origin xyz="-0.09998800046377702 9.147358505776733e-05 0.0008618985625794828" rpy="0 0 0"/>
@@ -52,12 +52,12 @@
     <origin xyz="0.08075 -0.000295 -0.109022" rpy="0 0 0"/>
     <geometry>
-      <mesh filename="file://$(find skid_steer_robot_description)/meshes/imu_1.stl" scale="0.001 0.001 0.001"/>
-    </geometry>
-    <material name="opaque170178196"/>
-  </visual>
-  <collision>
-    <origin xyz="0.08075 -0.000295 -0.109022" rpy="0 0 0"/>
-    <geometry>
-      <mesh filename="file://$(find skid_steer_robot_description)/meshes/imu_1.stl" scale="0.001 0.001 0.001"/>
+      <mesh filename="file://$(find skid_steer_robot_description)/meshes/imu.stl" scale="0.001 0.001 0.001"/>
+    </geometry>
+    <material name="opaque170178196"/>
+  </visual>
+  <collision>
+    <origin xyz="0.08075 -0.000295 -0.109022" rpy="0 0 0"/>
+    <geometry>
+      <mesh filename="file://$(find skid_steer_robot_description)/meshes/imu.stl" scale="0.001 0.001 0.001"/>
     </geometry>
   </collision>
@@ -166,10 +166,10 @@
   <origin xyz="-0.08075 0.000295 0.109022" rpy="0 0 0"/>
   <parent link="base_link"/>
-  <child link="lidar_1"/>
+  <child link="lidar"/>
 </joint>
 <joint name="imu_joint" type="fixed">
   <origin xyz="-0.08075 0.000295 0.109022" rpy="0 0 0"/>
   <parent link="base_link"/>
-  <child link="imu_1"/>
+  <child link="imu"/>
 </joint>
 <joint name="camera_joint" type="fixed">

Commit message: updated wheel mesh

File: skid_steer_robot_description/urdf/skid_steer_robot.xacro (robot description, xacro)
@@ -85,17 +85,17 @@
 <link name="right_front_wheel_1">
   <inertial>
-    <origin xyz="2.3498597991056247e-07 -0.03137906657473147 -4.712920191746184e-07" rpy="0 0 0"/>
-    <mass value="0.94911119349937"/>
-    <inertia ixx="0.001555" iyy="0.002702" izz="0.001555" ixy="0.0" iyz="-0.0" ixz="-0.0"/>
-  </inertial>
-  <visual>
-    <origin xyz="-0.10925 0.180205 -0.118022" rpy="0 0 0"/>
+    <origin xyz="8.243405957841787e-15 -0.032472752043596786 9.685754420729609e-10" rpy="0 0 0"/>
+    <mass value="8.688740501145128"/>
+    <inertia ixx="0.016085" iyy="0.027779" izz="0.016085" ixy="0.0" iyz="0.0" ixz="-0.0"/>
+  </inertial>
+  <visual>
+    <origin xyz="-0.19 0.1805 -0.08" rpy="0 0 0"/>
     <geometry>
       <mesh filename="file://$(find skid_steer_robot_description)/meshes/right_front_wheel_1.stl" scale="0.001 0.001 0.001"/>
     </geometry>
-    <material name="opaque170178196"/>
-  </visual>
-  <collision>
-    <origin xyz="-0.10925 0.180205 -0.118022" rpy="0 0 0"/>
+    <material name="steel_satin"/>
+  </visual>
+  <collision>
+    <origin xyz="-0.19 0.1805 -0.08" rpy="0 0 0"/>
     <geometry>
       <mesh filename="file://$(find skid_steer_robot_description)/meshes/right_front_wheel_1.stl" scale="0.001 0.001 0.001"/>
@@ -105,17 +105,17 @@
 <link name="right_back_wheel_1">
   <inertial>
-    <origin xyz="2.3498597973015123e-07 -0.03137906657473144 -4.712920194660519e-07" rpy="0 0 0"/>
-    <mass value="0.9491111934993678"/>
-    <inertia ixx="0.001555" iyy="0.002702" izz="0.001555" ixy="0.0" iyz="-0.0" ixz="-0.0"/>
-  </inertial>
-  <visual>
-    <origin xyz="0.27075 0.180205 -0.118022" rpy="0 0 0"/>
+    <origin xyz="8.243405957841787e-15 -0.032472752043596786 9.685754004395974e-10" rpy="0 0 0"/>
+    <mass value="8.688740501145128"/>
+    <inertia ixx="0.016085" iyy="0.027779" izz="0.016085" ixy="0.0" iyz="0.0" ixz="-0.0"/>
+  </inertial>
+  <visual>
+    <origin xyz="0.19 0.1805 -0.08" rpy="0 0 0"/>
     <geometry>
       <mesh filename="file://$(find skid_steer_robot_description)/meshes/right_back_wheel_1.stl" scale="0.001 0.001 0.001"/>
     </geometry>
-    <material name="opaque170178196"/>
-  </visual>
-  <collision>
-    <origin xyz="0.27075 0.180205 -0.118022" rpy="0 0 0"/>
+    <material name="steel_satin"/>
+  </visual>
+  <collision>
+    <origin xyz="0.19 0.1805 -0.08" rpy="0 0 0"/>
     <geometry>
       <mesh filename="file://$(find skid_steer_robot_description)/meshes/right_back_wheel_1.stl" scale="0.001 0.001 0.001"/>
@@ -125,17 +125,17 @@
 <link name="left_front_wheel_1">
   <inertial>
-    <origin xyz="-9.543055692895486e-09 0.03137930359057159 -1.2051076318797538e-07" rpy="0 0 0"/>
-    <mass value="0.9491110270115712"/>
-    <inertia ixx="0.001555" iyy="0.002702" izz="0.001555" ixy="-0.0" iyz="0.0" ixz="-0.0"/>
-  </inertial>
-  <visual>
-    <origin xyz="-0.10925 -0.180795 -0.118022" rpy="0 0 0"/>
+    <origin xyz="8.243405957841787e-15 0.032472752043596786 9.685754559507487e-10" rpy="0 0 0"/>
+    <mass value="8.688740501145128"/>
+    <inertia ixx="0.016085" iyy="0.027779" izz="0.016085" ixy="-0.0" iyz="-0.0" ixz="-0.0"/>
+  </inertial>
+  <visual>
+    <origin xyz="-0.19 -0.1805 -0.08" rpy="0 0 0"/>
     <geometry>
       <mesh filename="file://$(find skid_steer_robot_description)/meshes/left_front_wheel_1.stl" scale="0.001 0.001 0.001"/>
     </geometry>
-    <material name="opaque170178196"/>
-  </visual>
-  <collision>
-    <origin xyz="-0.10925 -0.180795 -0.118022" rpy="0 0 0"/>
+    <material name="steel_satin"/>
+  </visual>
+  <collision>
+    <origin xyz="-0.19 -0.1805 -0.08" rpy="0 0 0"/>
     <geometry>
       <mesh filename="file://$(find skid_steer_robot_description)/meshes/left_front_wheel_1.stl" scale="0.001 0.001 0.001"/>
@@ -145,17 +145,17 @@
 <link name="left_back_wheel_1">
   <inertial>
-    <origin xyz="-9.543055567995395e-09 0.03137930359057167 -1.2051076297980856e-07" rpy="0 0 0"/>
-    <mass value="0.9491110270115715"/>
-    <inertia ixx="0.001555" iyy="0.002702" izz="0.001555" ixy="-0.0" iyz="0.0" ixz="-0.0"/>
-  </inertial>
-  <visual>
-    <origin xyz="0.27075 -0.180795 -0.118022" rpy="0 0 0"/>
+    <origin xyz="8.243405957841787e-15 0.032472752043596786 9.685754420729609e-10" rpy="0 0 0"/>
+    <mass value="8.688740501145128"/>
+    <inertia ixx="0.016085" iyy="0.027779" izz="0.016085" ixy="0.0" iyz="0.0" ixz="0.0"/>
+  </inertial>
+  <visual>
+    <origin xyz="0.19 -0.1805 -0.08" rpy="0 0 0"/>
     <geometry>
       <mesh filename="file://$(find skid_steer_robot_description)/meshes/left_back_wheel_1.stl" scale="0.001 0.001 0.001"/>
     </geometry>
-    <material name="opaque170178196"/>
-  </visual>
-  <collision>
-    <origin xyz="0.27075 -0.180795 -0.118022" rpy="0 0 0"/>
+    <material name="steel_satin"/>
+  </visual>
+  <collision>
+    <origin xyz="0.19 -0.1805 -0.08" rpy="0 0 0"/>
     <geometry>
       <mesh filename="file://$(find skid_steer_robot_description)/meshes/left_back_wheel_1.stl" scale="0.001 0.001 0.001"/>
